Commit message: Ros2 for beginners level 2: Done

File: my_robot_description/urdf/common_properties.xacro (robot description, xacro)
@@ -6,4 +6,10 @@
     <material name="grey">
         <color rgba="0.5 0.5 0.5 1" />
+    </material>
+    <material name="orange">
+        <color rgba="1 0.65 0 1" />
+    </material>
+    <material name="yellow">
+        <color rgba="1 1 0 1" />
     </material>
     <xacro:macro name="box_inertia" params="m x y z o_xyz o_rpy">

File: my_robot_description/urdf/mobile_base.xacro (robot description, xacro)
@@ -62,4 +62,5 @@
             o_xyz="0 0 0" o_rpy="0 0 0"/>
     </link>
+    <!-- joints     -->
     <joint name="base_joint" type="fixed">
         <parent link="base_footprint" />

File: my_robot_description/urdf/my_robot.urdf.xacro (robot description, xacro)
@@ -5,3 +5,10 @@
     <xacro:include filename="mobile_base_gz.xacro"/>
     <xacro:include filename="camera.xacro"/>
+    <xacro:include filename="arm.xacro"/>
+    <xacro:robot_arm />
+    <joint name="base_arm_base_joint" type="fixed">
+        <parent link="base_link"/>
+        <child link="arm_base_link"/>
+        <origin xyz="${base_length/4.0} 0 ${base_height}" rpy="0 0 0"/>
+    </joint>
 </robot>
