Commit message: Fixed gazebo wrong direction; add correction factor to velocity, but still not good.

File: my_robot_description/urdf/mobile_base.xacro (robot description, xacro)
@@ -71,5 +71,5 @@
         <parent link="base_link" />
         <child link="right_wheel_link" />
-        <origin xyz="${-base_length/4.0} ${-(base_width+wheel_length)/2.0} 0" rpy="${pi/2.0} 0 0" />
+        <origin xyz="${-base_length/4.0} ${-(base_width+wheel_length)/2.0} 0" rpy="${-pi/2.0} 0 0" />
         <axis xyz="0 0 1"/>
     </joint>
@@ -77,5 +77,5 @@
         <parent link="base_link" />
         <child link="left_wheel_link" />
-        <origin xyz="${-base_length/4.0} ${(base_width+wheel_length)/2.0} 0" rpy="${pi/2.0} 0 0" />
+        <origin xyz="${-base_length/4.0} ${(base_width+wheel_length)/2.0} 0" rpy="${-pi/2.0} 0 0" />
         <axis xyz="0 0 1"/>
     </joint>
